File: pcb/logeek_mk2.kicad_pcb (KiCad board)
At the start: 2 copper layers, 68.6 x 53.3 mm, 132 parts, among them P1 Power, P10 DG301-2P 5.08mm, P11 BARREL_JACK, P12 USB_B, P13 DC3 5x2, P14 Power, P15 Analog, P16 Digital, P17 Digital, P2 Analog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

Commit message: Final revise before fabrication of Rev.B
Parts:
- removed the FID2 at (113.5, 76.8)
- L3: value DLW21SN900SQ2 -> DLW31SN222SQ2; footprint Logeek_MK2:CommonModeChoke_0805 -> Logeek_MK2:CommonModeChoke_1206
- renumbered FID3 to FID2
Routing:
- net +3V3: track 294.5 -> 292.8 mm
- net /DM: track 4.13 -> 3.35 mm
- net /DP: track 7.10 -> 6.42 mm
- net /USBDM: track 16.3 -> 15.8 mm
- net (no net): vias 1 -> 0
Other:
- board text added: "+4.5V~~+24V"
- board text removed: "+5V~~+24V"

Commit message: Annotation update.
Parts:
- D5: value LED GREEN -> LED
- D6: value TVS 10 V -> TVS
- FB1, FB2, FB3, FB4, FB5: value FILTER -> Ferrite
- FID1, FID2: value Fiducial_1mm_Dia_2.54mm_Outer_CopperTop -> F
- P11: value BARREL_JACK -> Barrel Jack
- P14: value Power -> Digital
- P5, P6, P7, P8: value CONN_1 -> MH
