File: pcb/logeek_mk2.sch (KiCad schematic (older format))
At the start: 127 parts, among them P1 Power, P10 DG301-2P 5.08mm, P11 BARREL_JACK, P12 USB_B, P13 DC3 5x2, P14 Power, P15 Analog, P16 Digital, P17 Digital, P2 Analog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

Commit message: Annotation update.
Parts:
- D5: value LED GREEN -> LED
- D6: value TVS 10 V -> TVS
- FB1, FB2, FB3, FB4, FB5: value FILTER -> Ferrite
- P11: value BARREL_JACK -> Barrel Jack
- P14: value Power -> Digital
- P5, P6, P7, P8: value CONN_1 -> MH
Changed lines of the file:
@@
 P 15700 675
 F 0 "P5" H 15780 675 40  0000 L CNN
-F 1 "CONN_1" H 15700 730 30  0001 C CNN
+F 1 "MH" H 15700 730 30  0001 C CNN
 F 2 "Logeek_MK2:Arduino_1pin" H 15700 675 60  0001 C CNN
 F 3 "" H 15700 675 60  0000 C CNN
@@
 P 15775 675
 F 0 "P6" H 15855 675 40  0000 L CNN
-F 1 "CONN_1" H 15775 730 30  0001 C CNN
+F 1 "MH" H 15775 730 30  0001 C CNN
 F 2 "Logeek_MK2:Arduino_1pin" H 15775 675 60  0001 C CNN
 F 3 "" H 15775 675 60  0000 C CNN
@@
 P 15850 675
 F 0 "P7" H 15930 675 40  0000 L CNN
-F 1 "CONN_1" H 15850 730 30  0001 C CNN
+F 1 "MH" H 15850 730 30  0001 C CNN
 F 2 "Logeek_MK2:Arduino_1pin" H 15850 675 60  0001 C CNN
 F 3 "" H 15850 675 60  0000 C CNN
@@
 P 15925 675
 F 0 "P8" H 16005 675 40  0000 L CNN
-F 1 "CONN_1" H 15925 730 30  0001 C CNN
+F 1 "MH" H 15925 730 30  0001 C CNN
 F 2 "Logeek_MK2:Arduino_1pin" H 15925 675 60  0001 C CNN
 F 3 "" H 15925 675 60  0000 C CNN
@@
 P 2550 2250
 F 0 "FB4" H 2550 2400 50  0000 C CNN
-F 1 "FILTER" H 2550 2150 50  0000 C CNN
+F 1 "Ferrite" H 2550 2150 50  0000 C CNN
 F 2 "Resistors_SMD:R_0603" H 2550 2250 60  0001 C CNN
 F 3 "" H 2550 2250 60  0000 C CNN
@@
 P 1350 3750
 F 0 "FB2" H 1350 3900 50  0000 C CNN
-F 1 "FILTER" H 1350 3650 50  0000 C CNN
+F 1 "Ferrite" H 1350 3650 50  0000 C CNN
 F 2 "Resistors_SMD:R_0603" H 1350 3750 60  0001 C CNN
 F 3 "" H 1350 3750 60  0000 C CNN
@@
 P 2000 5150
 F 0 "FB3" H 2000 5300 50  0000 C CNN
-F 1 "FILTER" H 2000 5050 50  0000 C CNN
+F 1 "Ferrite" H 2000 5050 50  0000 C CNN
 F 2 "Resistors_SMD:R_0603" H 2000 5150 60  0001 C CNN
 F 3 "" H 2000 5150 60  0000 C CNN
@@
 P 1350 3050
 F 0 "FB1" H 1350 3200 50  0000 C CNN
-F 1 "FILTER" H 1350 2950 50  0000 C CNN
+F 1 "Ferrite" H 1350 2950 50  0000 C CNN
 F 2 "Resistors_SMD:R_0603" H 1350 3050 60  0001 C CNN
 F 3 "" H 1350 3050 60  0000 C CNN
@@
 P 10600 4650
 F 0 "FB5" H 10600 4800 50  0000 C CNN
-F 1 "FILTER" H 10600 4550 50  0000 C CNN
+F 1 "Ferrite" H 10600 4550 50  0000 C CNN
 F 2 "Resistors_SMD:R_0603" H 10600 4650 60  0001 C CNN
 F 3 "" H 10600 4650 60  0000 C CNN
@@
 P 12850 8850
 F 0 "D5" H 12850 8950 50  0000 C CNN
-F 1 "LED GREEN" H 12850 8700 50  0000 C CNN
+F 1 "LED" H 12850 8700 50  0000 C CNN
 F 2 "Logeek_MK2:LED-0603" H 12850 8850 60  0001 C CNN
 F 3 "" H 12850 8850 60  0000 C CNN
@@
 P 14550 8500
 F 0 "P14" V 14500 8500 60  0000 C CNN
-F 1 "Power" V 14600 8500 60  0000 C CNN
+F 1 "Digital" V 14600 8500 60  0000 C CNN
 F 2 "Logeek_MK2:Socket_Strip_Arduino_1x08" H 14550 8500 60  0001 C CNN
 F 3 "" H 14550 8500 60  0000 C CNN
@@
 P 1300 10450
 F 0 "P11" H 1200 10700 60  0000 C CNN
-F 1 "BARREL_JACK" H 1300 10250 60  0001 C CNN
+F 1 "Barrel Jack" H 1300 10250 60  0001 C CNN
 F 2 "Logeek_MK2:BARREL_JACK" H 1300 10450 60  0001 C CNN
 F 3 "" H 1300 10450 60  0000 C CNN
@@
 P 1300 9100
 F 0 "D6" H 1150 9200 50  0000 C CNN
-F 1 "TVS 10 V" H 1350 9000 50  0000 C CNN
+F 1 "TVS" H 1350 9000 50  0000 C CNN
 F 2 "Resistors_SMD:R_0402_HandSoldering" H 1300 9100 60  0001 C CNN
 F 3 "" H 1300 9100 60  0000 C CNN
@@
 00 39 19 59 AF 35 42 7E F6 69 BC 65 B4 12 E9 FA 23 84 AE 83 6F 0F D1 9A 40 57 B7 F2 6C 29 EA 3A
 9E 6A A1 85 FF 38 9C BE D1 9C BA 77 9F E3 4F 15 EE 64 AF AB 31 A7 47 CD F6 48 3D E9 C1 75 26 7B
-81 F3 EA B7 E7 8B FF 0F 20 F4 78 B9 DD 14 EB 4B 00 00 00 00 49 45 4E 44 AE 42 60 82 8E
+81 F3 EA B7 E7 8B FF 0F 20 F4 78 B9 DD 14 EB 4B 00 00 00 00 49 45 4E 44 AE 42 60 82 BF
 EndData
 $EndBitmap
